File: kicad/Ethernet-SchDoc.sch (KiCad schematic (older format))
At the start: 89 parts, among them IC1 VSC8541XMV-01, J12 RJHSE5384, T1 TG111-MSC13LF, U35 MIC5353-2.5YMT-TR, U36 NCP133AMX100TCG, U37 SN74AUP1T34DCKR, U38 SN74AUP1T34DCKR, Y3 25 MHz

Commit message: Ki5 update
Parts:
- removed TP4, TP5, TP6: ~, symbol HiFiveUnleashed:Testpoint
- added TP4, TP5, TP6: Test_Point, TestPoint:TestPoint_Pad_D1.0mm, symbol Connector:Test_Point
- C178, C179, C181, C182, C183, C186, C188, C189, C190, C191, C192, C193, C194, C195, C197, C198, C199, C200, C201, C202, C205, C208, C209, C210, C211, C212, C213, C214, C215, C216, C217: footprint (none) -> Capacitor_SMD:C_0402_1005Metric
- C180, C184, C185, C187, C196: footprint (none) -> Capacitor_SMD:C_0603_1608Metric
- C203, C204: footprint (none) -> Capacitor_SMD:C_1206_3216Metric
- FB3, FB4: footprint (none) -> Inductor_SMD:L_0402_1005Metric; symbol HiFiveUnleashed:Ferrite_Bead -> Device:Ferrite_Bead
- IC1: footprint (none) -> Package_DFN_QFN:QFN-68-1EP_8x8mm_Pitch0.4mm
- J12: footprint (none) -> Connector_RJ:RJ45_Amphenol_RJHSE538X
- R100, R101, R102, R103, R104, R105, R106, R107, R108, R109, R110, R111, R112, R113, R114, R115, R116, R79, R81, R83, R84, R86, R87, R88, R89, R90, R91, R92, R93, R94, R95, R96, R97, R98, R99: footprint (none) -> Resistor_SMD:R_0402_1005Metric
- R80, R82, R85: footprint (none) -> Resistor_SMD:R_Array_Concave_4x0402
- T1: symbol HiFiveUnleashed:GBE_TRANSFORMER -> Transformer:TG111-MSC13LF
- U35: symbol HiFiveUnleashed:MIC5353 -> Regulator_Linear:MIC5353-2.5YMT
- U36: symbol HiFiveUnleashed:NCP133 -> Regulator_Linear:NCP133AMX100TCG
- U37, U38: footprint (none) -> Package_TO_SOT_SMD:SOT-353_SC-70-5
- Y3: footprint (none) -> Crystal:Crystal_SMD_SeikoEpson_FA238-4Pin_3.2x2.5mm; symbol HiFiveUnleashed:XTAL_4p -> Device:Crystal_GND2
Connections:
- net labels added: +1V0, +1V8, +2V5, +3V3, +5V
- net labels removed: VDD
- wire segments 341 -> 345
- no-connect marks 0 -> 3
