File: kicad/FMC-SchDoc.sch (KiCad schematic (older format))
At the start: 16 parts, among them J9 FMC-HPC, J9_10 FMC-HPC, J9_2 FMC-HPC, J9_3 FMC-HPC, J9_4 FMC-HPC, J9_5 FMC-HPC, J9_6 FMC-HPC, J9_7 FMC-HPC, J9_8 FMC-HPC, J9_9 FMC-HPC, U49 DNP

Commit message: Ki5 update
Parts:
- removed J9: FMC-HPC, symbol HiFiveUnleashed:FMC-HPC_1
- removed J9_10: FMC-HPC, symbol HiFiveUnleashed:FMC-HPC_10
- removed J9_2: FMC-HPC, symbol HiFiveUnleashed:FMC-HPC_2
- removed J9_3: FMC-HPC, symbol HiFiveUnleashed:FMC-HPC_3
- removed J9_4: FMC-HPC, symbol HiFiveUnleashed:FMC-HPC_4
- removed J9_5: FMC-HPC, symbol HiFiveUnleashed:FMC-HPC_5
- removed J9_6: FMC-HPC, symbol HiFiveUnleashed:FMC-HPC_6
- removed J9_7: FMC-HPC, symbol HiFiveUnleashed:FMC-HPC_7
- removed J9_8: FMC-HPC, symbol HiFiveUnleashed:FMC-HPC_8
- removed J9_9: FMC-HPC, symbol HiFiveUnleashed:FMC-HPC_9
- removed U49: DNP, symbol HiFiveUnleashed:M24C02_SO8
- added J9: ASP-134602-01, symbol Connector:ASP-134602-01
- added U49: M24C02-WMN, Package_SO:TSSOP-8_4.4x3mm_P0.65mm, symbol Memory_EEPROM:M24C02-WDW
- C267: footprint (none) -> Capacitor_SMD:C_0402_1005Metric
- R172, R173, R174, R175: footprint (none) -> Resistor_SMD:R_0402_1005Metric
Connections:
- net labels added: +12V, +1V8, +3.3VP
- net labels removed: 3P3VAUX, VDD
- wire segments 423 -> 422
- no-connect marks 0 -> 159
