File: kicad/FT2232-SchDoc.sch (KiCad schematic (older format))
At the start: 49 parts, among them J7 MicroUSB2.0 Connector, U13 FT2232HL, U28 SN74AUP1T34DCKR, U29 SN74AUP1T34DCKR, U30 SN74AUP1T34DCKR, U31 SN74AUP1T34DCKR, U32 SN74AUP1T34DCKR, U33 SN74AUP1T34DCKR, Y2 12 MHz

Commit message: Ki5 update
Parts:
- removed J7: MicroUSB2.0 Connector, symbol HiFiveUnleashed:MicroUSB2.0_Connector
- removed Q4_2: ~, symbol HiFiveUnleashed:FDG6335N_1
- added J7: USB_B_Micro, symbol Connector:USB_B_Micro
- added Q4: FDG6335N, Package_TO_SOT_SMD:SOT-363_SC-70-6, symbol Transistor_FET:FDG6335N
- C100, C101, C102, C103, C104, C105, C106, C107, C108, C109, C110, C112, C113, C114, C115, C166, C167, C168, C169, C170, C171, C172, C173, C174, C175, C176, C177: footprint (none) -> Capacitor_SMD:C_0402_1005Metric
- C111: footprint (none) -> Capacitor_SMD:C_0603_1608Metric
- D5, D6: footprint (none) -> Diode_SMD:D_0603_1608Metric
- FB1, FB2: footprint (none) -> Inductor_SMD:L_0402_1005Metric; symbol HiFiveUnleashed:Ferrite_Bead -> Device:Ferrite_Bead
- R23, R26, R31, R32, R33, R34, R74: footprint (none) -> Resistor_SMD:R_0402_1005Metric
- U13: footprint (none) -> Package_QFP:LQFP-64_10x10mm_P0.5mm
- U28, U29, U30, U31, U32, U33: footprint (none) -> Package_TO_SOT_SMD:SOT-353_SC-70-5
- Y2: footprint (none) -> Crystal:Crystal_SMD_Abracon_ABM8G-4Pin_3.2x2.5mm; symbol HiFiveUnleashed:XTAL_4p -> Device:Crystal_GND2
Connections:
- net labels added: +1V8, +3V3, VDDA
- net labels removed: VBUS, VCORE_FT, VTT
- wire segments 137 -> 132
- no-connect marks 0 -> 31
