File: kicad/FT2232-SchDoc.sch (KiCad schematic (older format))
At the start: 49 parts, among them J7 USB_B_Micro, Q4 FDG6335N, U13 FT2232HL, U28 SN74AUP1T34DCKR, U29 SN74AUP1T34DCKR, U30 SN74AUP1T34DCKR, U31 SN74AUP1T34DCKR, U32 SN74AUP1T34DCKR, U33 SN74AUP1T34DCKR, Y2 12 MHz

Commit message: ki5 update
Parts:
- J7: footprint (none) -> Connector_USB:USB_Micro-B_Molex_47346-0001
Changed lines of the file:
@@
 EESchema Schematic File Version 4
-LIBS:Ki5-cache
 EELAYER 26 0
 EELAYER END
@@
 encoding utf-8
 Sheet 6 9
-Title "U540 RISC-V MPU eval board"
+Title "USB to UART and JTAG"
 Date "08 05 2018"
 Rev ""
 Comp ""
-Comment1 "USB to UART and JTAG"
+Comment1 ""
 Comment2 ""
 Comment3 ""
@@
 F 0 "J7" H 2505 5917 50  0000 C CNN
 F 1 "USB_B_Micro" H 2505 5826 50  0000 C CNN
-F 2 "" H 2600 5400 50  0001 C CNN
+F 2 "Connector_USB:USB_Micro-B_Molex_47346-0001" H 2600 5400 50  0001 C CNN
 F 3 "~" H 2600 5400 50  0001 C CNN
 	1    2450 5450
