File: kicad/Freedom-U540_2-SchDoc.sch (KiCad schematic (older format))
At the start: 136 parts, among them J1 96BoardsLowSpeedExpansion, J10 MicroSD_CD, J11 Header 2x5, J13 Header 2x4, J2 Header 2x10, U12 256Mbit, U1_4 FU540-C000, U1_5 FU540-C000, U1_6 FU540-C000, U20 SN74AUP1T34DCKR, U21 SN74AUP1T34DCKR, U22 SN74AUP1T34DCKR, U23 SN74AUP1T34DCKR, U24 SN74AUP1T34DCKR, U25 SN74AUP1T34DCKR, U26 TPD6F003DQDR, X1 33.3333 MHz, X2 1.0 MHz, Y1 33.333 MHz

Commit message: Ki5 update
Parts:
- removed J1: 96BoardsLowSpeedExpansion, symbol HiFiveUnleashed:96BoardsLowSpeedExpansion
- removed J10: MicroSD_CD, symbol HiFiveUnleashed:MicroSD_CD
- removed J11: Header 2x5, symbol HiFiveUnleashed:Header_2x5
- removed J13: Header 2x4, symbol HiFiveUnleashed:Header_2x4
- removed J2: Header 2x10, symbol HiFiveUnleashed:Header_2x10
- removed J3, J4, J5, J6: ~, symbol HiFiveUnleashed:MMCX_Connector
- removed Q1, Q2: ~, symbol HiFiveUnleashed:FDG6335N_1
- removed Q1_2, Q2_2, Q4: ~, symbol HiFiveUnleashed:FDG6335N_2
- removed Q6: ~, symbol HiFiveUnleashed:MOSFET-P_SOT23
- removed S2: SW-PB 4P, symbol HiFiveUnleashed:SW-PB_4P
- removed U12: 256Mbit, symbol HiFiveUnleashed:QuadSPI_SO16
- removed U1_4: FU540-C000, symbol HiFiveUnleashed:Freedom-U540_FCBGA_4
- removed U1_5: FU540-C000, symbol HiFiveUnleashed:Freedom-U540_FCBGA_6
- removed U1_6: FU540-C000, symbol HiFiveUnleashed:Freedom-U540_FCBGA_5
- removed U26: TPD6F003DQDR, symbol HiFiveUnleashed:TPD6F003DQDR
- added J1: Conn_02x20_Odd_Even, symbol Connector_Generic:Conn_02x20_Odd_Even
- added J10: Micro_SD_Card_Det, symbol Connector:Micro_SD_Card_Det
- added J11: Conn_02x05_Odd_Even, symbol Connector_Generic:Conn_02x05_Odd_Even
- added J13: Conn_02x04_Odd_Even, symbol Connector_Generic:Conn_02x04_Odd_Even
- added J2: Conn_02x10_Odd_Even, symbol Connector_Generic:Conn_02x10_Odd_Even
- added J3, J4, J5, J6: Conn_Coaxial, symbol Connector:Conn_Coaxial
- added Q1, Q2, Q4: FDG6335N, Package_TO_SOT_SMD:SOT-363_SC-70-6, symbol Transistor_FET:FDG6335N
- added Q6: IRLML6402, Package_TO_SOT_SMD:SOT-23, symbol Transistor_FET:IRLML6402
- added S2: SW_Push, Button_Switch_SMD:SW_SPST_PTS645, symbol Switch:SW_Push
- added U1: FU540-C000, Package_BGA:BGA-484_23.0x23.0mm_Layout22x22_P1.0mm, symbol MCU_SiFive:FU540-C000
- added U12: IS25WP256D, Package_SO:SOIC-16W_7.5x10.3mm_P1.27mm, symbol Memory_Flash:IS25WP256D
- added U26: TPD6F003, symbol Power_Protection:TPD6F003
- C130, C131, C132, C133, C134, C135, C136, C137, C138, C153, C154, C155, C156, C157, C158, C159, C160, C161, C162, C163, C164, C165, C206, C207, C241, C242, C243, C244, C245, C246, C247, C248, C249, C250, C251, C252, C253, C254, C255, C256, C257, C258: footprint (none) -> Capacitor_SMD:C_0402_1005Metric
- D1, D2, D3, D4: footprint (none) -> LED_SMD:LED_0603_1608Metric; symbol HiFiveUnleashed:LED -> Device:LED
- D10, D11: footprint (none) -> Diode_SMD:D_0603_1608Metric
- R12, R13, R139, R14, R140, R141, R142, R143, R144, R15, R16, R160, R161, R162, R17, R18, R182, R183, R186, R19, R20, R21, R22, R24, R25, R27, R28, R29, R30, R37, R44, R45, R46, R47, R48, R49, R50, R51, R52, R53, R54, R55, R56, R57, R58, R59, R65, R72, R73: footprint (none) -> Resistor_SMD:R_0402_1005Metric
- R158, R159: footprint (none) -> Resistor_SMD:R_Array_Concave_4x0402
- RS10, RS7, RS8, RS9: symbol HiFiveUnleashed:Resistor_4p -> Device:R_Shunt
- S1, S3: footprint (none) -> Button_Switch_SMD:SW_DIP_SPSTx06_Slide_6.7x16.8mm_W8.61mm_P2.54mm_LowProfile; symbol HiFiveUnleashed:SW_DIP-6 -> Switch:SW_DIP_x06
- U20, U21, U22, U23, U24, U25: footprint (none) -> Package_TO_SOT_SMD:SOT-353_SC-70-5
- X1: footprint (none) -> Oscillator:Oscillator_SMD_EuroQuartz_XO32-4Pin_3.2x2.5mm; symbol HiFiveUnleashed:OSC_4P_OE -> Oscillator:XO32
- X2: footprint (none) -> Oscillator:Oscillator_SMD_EuroQuartz_XO32-4Pin_3.2x2.5mm; symbol HiFiveUnleashed:OSC_SiTime_OE -> Oscillator:XO32
- Y1: footprint (none) -> Crystal:Crystal_SMD_3225-4Pin_3.2x2.5mm; symbol HiFiveUnleashed:XTAL_4p -> Device:Crystal_GND2
Connections:
- net labels added: +12V, +1V1, +1V8, +3.3VA, +3V3, +5V, VCOM
- wire segments 827 -> 811
- no-connect marks 0 -> 13
