File: kicad/Freedom-U540_2-SchDoc.sch (KiCad schematic (older format))
At the start: 132 parts, among them J1 Conn_02x20_Odd_Even, J10 Micro_SD_Card_Det, J11 Conn_02x05_Odd_Even, J13 Conn_02x04_Odd_Even, J2 Conn_02x10_Odd_Even, J3 Conn_Coaxial, J4 Conn_Coaxial, J5 Conn_Coaxial, J6 Conn_Coaxial, Q1 FDG6335N, Q2 FDG6335N, Q4 FDG6335N, Q6 IRLML6402, U1 FU540-C000, U12 IS25WP256D, U20 SN74AUP1T34DCKR, U21 SN74AUP1T34DCKR, U22 SN74AUP1T34DCKR, U23 SN74AUP1T34DCKR, U24 SN74AUP1T34DCKR, U25 SN74AUP1T34DCKR, U26 TPD6F003, X1 33.3333 MHz, X2 1.0 MHz, Y1 33.333 MHz

Commit message: ki5 update
Parts:
- added J14: Conn_02x11_Odd_Even, Connector_PinHeader_1.27mm:PinHeader_2x11_P1.27mm_Vertical_SMD, symbol Connector_Generic:Conn_02x11_Odd_Even
- J1: footprint (none) -> Connector_PinSocket_2.00mm:PinSocket_2x20_P2.00mm_Vertical_SMD
- J10: footprint (none) -> Connector_Card:microSD_HC_Hirose_DM3D-SF
- J11: footprint (none) -> Connector_PinHeader_1.27mm:PinHeader_2x05_P1.27mm_Vertical_SMD
- J13: footprint (none) -> Connector_PinHeader_1.27mm:PinHeader_2x04_P1.27mm_Vertical_SMD
- J2: footprint (none) -> Connector_PinSocket_2.00mm:PinSocket_2x10_P2.00mm_Vertical_SMD
- J3, J4, J5, J6: footprint (none) -> Connector_Coaxial:MMCX_Molex_73415-1471_Vertical
- RS10: footprint (none) -> Resistor_SMD:R_Shunt_Vishay_WSKW0612
- RS7, RS8, RS9: footprint (none) -> Resistor_SMD:R_0603_1608Metric; symbol Device:R_Shunt -> Device:R
- U26: footprint (none) -> Package_SON:WSON-12-1EP_1.35x2.5mm_P0.4mm_EP0.4x2mm
Connections:
- net labels added: AVDD_DDRPLL_N, AVDD_DDRPLL_P, VDD_DDRPLL_N, VDD_DDRPLL_P, VDD_DDR_MEM_N, VDD_DDR_MEM_P, VDD_DDR_SOC_N, VDD_DDR_SOC_P, VDD_GEMGXLPLL_N, VDD_GEMGXLPLL_P, VDD_GIVDD_N, VDD_GIVDD_P
- wire segments 811 -> 835
