File: kicad/Power-SchDoc.sch (KiCad schematic (older format))
At the start: 77 parts, among them J8 PowerJack2P_SH, U14 TLV62080DSGR, U15 TLV62084DSGT, U16 TLV62095RGTR, U17 LP5907MFX-1.8/NOPB, U18 TPS51363, U19 LM3880MFE-1AA/NOPB, U27 TPS62133RGTT, U50 TLV62080DSGR

Commit message: Ki5 update
Parts:
- removed J19: ~, symbol HiFiveUnleashed:PC_FAN_3P
- removed J8: PowerJack2P_SH, symbol HiFiveUnleashed:PowerJack2P_SH
- removed M1, M2, M3, M4, M5, M6: ~, symbol HiFiveUnleashed:M2.5
- removed Q5: ~, symbol HiFiveUnleashed:FDG6335N_2
- removed Q5_2: ~, symbol HiFiveUnleashed:FDG6335N_1
- removed S4: ~, symbol HiFiveUnleashed:SW-SPDT
- added J19: Fan_Tacho, Connector:FanPinHeader_1x03_P2.54mm_Vertical, symbol Motor:Fan_Tacho
- added J8: Jack-DC, symbol Connector:Jack-DC
- added M1, M2, M3, M4, M5, M6: Mounting_Hole_PAD, MountingHole:MountingHole_2.7mm_M2.5_ISO7380_Pad, symbol Mechanical:Mounting_Hole_PAD
- added Q5: FDG6335N, Package_TO_SOT_SMD:SOT-363_SC-70-6, symbol Transistor_FET:FDG6335N
- added S4: SW_Push_SPDT, symbol Switch:SW_Push_SPDT
- C116, C117, C121, C124, C139, C140, C141, C149, C219, C281: footprint (none) -> Capacitor_SMD:C_0805_2012Metric
- C118, C119, C142, C143, C144, C145, C146, C147, C148, C151, C152, C220: footprint (none) -> Capacitor_SMD:C_0402_1005Metric
- C120, C122, C218: footprint (none) -> Capacitor_SMD:C_0603_1608Metric
- C150: footprint (none) -> Capacitor_Tantalum_SMD:CP_EIA-7343-20_Kemet-V
- D12: footprint (none) -> Diode_SMD:D_0603_1608Metric
- D7, D8: footprint (none) -> Diode_SMD:D_SOD-123F
- D9: footprint (none) -> LED_SMD:LED_0603_1608Metric; symbol HiFiveUnleashed:LED -> Device:LED
- L1, L2, L3, L6: footprint (none) -> Inductor_SMD:L_Wuerth_MAPI-2512; symbol HiFiveUnleashed:Inductor -> Device:L
- L4: footprint (none) -> Inductor_SMD:L_Wuerth_MAPI-2510; symbol HiFiveUnleashed:Inductor -> Device:L
- L5: symbol HiFiveUnleashed:Inductor -> Device:L
- R117, R138, R156, R177, R35, R36, R38, R39, R40, R41, R42, R43, R60, R61, R62, R63, R64, R66, R67, R68, R69, R71: footprint (none) -> Resistor_SMD:R_0402_1005Metric
- U14, U50: value TLV62080DSGR -> TLV62080DSGx; footprint (none) -> Package_SON:WSON-8-1EP_2x2mm_P0.5mm_EP0.9x1.6mm; symbol HiFiveUnleashed:TLV6208x -> Regulator_Switching:TLV62080DSGx
- U15: value TLV62084DSGT -> TLV62084DSGx; footprint (none) -> Package_SON:WSON-8-1EP_2x2mm_P0.5mm_EP0.9x1.6mm; symbol HiFiveUnleashed:TLV6208x -> Regulator_Switching:TLV62080DSGx
- U16: footprint (none) -> Package_DFN_QFN:QFN-16-1EP_3x3mm_P0.5mm_EP1.8x1.8mm; symbol HiFiveUnleashed:TLV62095 -> Regulator_Switching:TLV62095RGTx
- U17: footprint (none) -> Package_TO_SOT_SMD:SOT-23-5; symbol HiFiveUnleashed:LP5907MFX -> Regulator_Linear:LP5907MFX-1.8
- U18: symbol HiFiveUnleashed:TPS51363 -> Regulator_Switching:TPS51363
- U19: footprint (none) -> Package_TO_SOT_SMD:SOT-23-6
- U27: footprint (none) -> Package_DFN_QFN:QFN-16-1EP_3x3mm_P0.5mm_EP1.8x1.8mm; symbol HiFiveUnleashed:TPS6213x -> Regulator_Switching:TPS62133
Connections:
- net labels added: +12V, +1V1, +1V8, +3V3, +5V, +VSW, VCOM, VMEM
- wire segments 278 -> 284
- no-connect marks 0 -> 6
