File: kicad/Power-SchDoc.sch (KiCad schematic (older format))
At the start: 76 parts, among them J19 Fan_Tacho, J8 Jack-DC, M1 Mounting_Hole_PAD, M2 Mounting_Hole_PAD, M3 Mounting_Hole_PAD, M4 Mounting_Hole_PAD, M5 Mounting_Hole_PAD, M6 Mounting_Hole_PAD, Q5 FDG6335N, U14 TLV62080DSGx, U15 TLV62084DSGx, U16 TLV62095RGTR, U17 LP5907MFX-1.8/NOPB, U18 TPS51363, U19 LM3880MFE-1AA/NOPB, U27 TPS62133RGTT, U50 TLV62080DSGx

Commit message: ki5 update
Parts:
- J8: footprint (none) -> Connector_BarrelJack:BarrelJack_CUI_PJ-063BH_Horizontal
- L5: footprint (none) -> Inductor_SMD:L_Bourns_SRN6045TA
- S4: footprint (none) -> Button_Switch_THT:SW_NKK_BB15AH
- U18: footprint (none) -> Package_DFN_QFN:R-VFQFN-28-1EP_3.5x4.5mm_P0.4mm_EP2.1x3.1mm
Changed lines of the file:
@@
 EESchema Schematic File Version 4
-LIBS:Ki5-cache
 EELAYER 26 0
 EELAYER END
@@
 encoding utf-8
 Sheet 7 9
-Title "U540 RISC-V MPU eval board"
+Title "Power Supply"
 Date "08 05 2018"
 Rev ""
 Comp ""
-Comment1 "Power Supply"
+Comment1 ""
 Comment2 ""
 Comment3 ""
@@
 F 0 "L5" V 12295 5065 60  0000 L BNN
 F 1 "1.0uH" V 12300 4485 60  0000 L BNN
-F 2 "" H 12220 4670 60  0001 C CNN
+F 2 "Inductor_SMD:L_Bourns_SRN6045TA" H 12220 4670 60  0001 C CNN
 F 3 "" H 12220 4670 60  0000 C CNN
 F 4 "" H 320 100 50  0001 C CNN "ClassName"
@@
 F 0 "U18" H 10285 6845 50  0000 C CNN
 F 1 "TPS51363" H 10410 4745 50  0000 C CNN
-F 2 "" H 10600 3900 60  0001 C CNN
+F 2 "Package_DFN_QFN:R-VFQFN-28-1EP_3.5x4.5mm_P0.4mm_EP2.1x3.1mm" H 10600 3900 60  0001 C CNN
 F 3 "" H 10600 3900 60  0000 C CNN
 F 4 "" H 400 800 50  0001 C CNN "ClassName"
@@
 F 0 "J8" H 1878 1825 50  0000 C CNN
 F 1 "Jack-DC" H 1878 1734 50  0000 C CNN
-F 2 "" H 1850 1460 50  0001 C CNN
+F 2 "Connector_BarrelJack:BarrelJack_CUI_PJ-063BH_Horizontal" H 1850 1460 50  0001 C CNN
 F 3 "~" H 1850 1460 50  0001 C CNN
 	1    1800 1500
@@
 F 0 "S4" H 2100 4385 50  0000 C CNN
 F 1 "SW_Push_SPDT" H 2100 4294 50  0000 C CNN
-F 2 "" H 2100 4100 50  0001 C CNN
+F 2 "Button_Switch_THT:SW_NKK_BB15AH" H 2100 4100 50  0001 C CNN
 F 3 "" H 2100 4100 50  0001 C CNN
 	1    2100 4100
