File: kicad/DDR4_x8_32b_1-SchDoc.sch (KiCad schematic (older format))
At the start: 86 parts, among them U11 TPS51200DRC, U2 H5AN8G8NAFR-UH, U3 H5AN8G8NAFR-UH, U4 H5AN8G8NAFR-UH, U5 H5AN8G8NAFR-UH

Commit message: ki5 update
Parts:
- RS1: footprint (none) -> Resistor_SMD:R_Shunt_Vishay_WSKW0612
- RS11: footprint (none) -> Resistor_SMD:R_0603_1608Metric; symbol Device:R_Shunt -> Device:R; CrossRef 1, 4 -> 9
- U2, U3, U4, U5: footprint (none) -> Package_BGA:FBGA-78_7.5x11mm_Layout2x3x13_P0.8mm
Changed lines of the file:
@@
 EESchema Schematic File Version 4
-LIBS:Ki5-cache
 EELAYER 26 0
 EELAYER END
@@
 encoding utf-8
 Sheet 4 9
-Title "U540 RISC-V MPU eval board"
+Title "DDR4x8 32 Bits"
 Date "08 05 2018"
 Rev ""
 Comp ""
-Comment1 "DDR4x8 32 Bits"
+Comment1 ""
 Comment2 ""
 Comment3 ""
@@
 	4150 3400 4150 3300
 Wire Wire Line
-	11550 15200 10100 15200
-Wire Wire Line
 	19050 7000 18850 7000
 Wire Wire Line
@@
 F 0 "RS1" V 10180 14665 60  0000 R BNN
 F 1 "0R001" V 10185 14130 60  0000 R BNN
-F 2 "" H 10105 14200 60  0001 C CNN
+F 2 "Resistor_SMD:R_Shunt_Vishay_WSKW0612" H 10105 14200 60  0001 C CNN
 F 3 "" H 10105 14200 60  0000 C CNN
 F 4 "" H -145 100 50  0001 C CNN "ClassName"
@@
 F 0 "U5" H 11900 12965 50  0000 C CNN
 F 1 "H5AN8G8NAFR-UH" H 12455 8335 50  0000 C CNN
-F 2 "" H 12480 6050 60  0001 C CNN
+F 2 "Package_BGA:FBGA-78_7.5x11mm_Layout2x3x13_P0.8mm" H 12480 6050 60  0001 C CNN
 F 3 "" H 12480 6050 60  0000 C CNN
 F 4 "" H 630 2250 50  0001 C CNN "ClassName"
@@
 F 0 "U4" H 4820 12960 50  0000 C CNN
 F 1 "H5AN8G8NAFR-UH" H 5360 8340 50  0000 C CNN
-F 2 "" H 5400 6050 60  0001 C CNN
+F 2 "Package_BGA:FBGA-78_7.5x11mm_Layout2x3x13_P0.8mm" H 5400 6050 60  0001 C CNN
 F 3 "" H 5400 6050 60  0000 C CNN
 F 4 "" H 650 2250 50  0001 C CNN "ClassName"
@@
 F 0 "U3" H 11905 6750 50  0000 C CNN
 F 1 "H5AN8G8NAFR-UH" H 12485 2140 50  0000 C CNN
-F 2 "" H 12495 -150 60  0001 C CNN
+F 2 "Package_BGA:FBGA-78_7.5x11mm_Layout2x3x13_P0.8mm" H 12495 -150 60  0001 C CNN
 F 3 "" H 12495 -150 60  0000 C CNN
 F 4 "" H 645 2250 50  0001 C CNN "ClassName"
@@
 F 0 "U2" H 4610 6745 50  0000 C CNN
 F 1 "H5AN8G8NAFR-UH" H 5175 2150 50  0000 C CNN
-F 2 "" H 5200 -150 60  0001 C CNN
+F 2 "Package_BGA:FBGA-78_7.5x11mm_Layout2x3x13_P0.8mm" H 5200 -150 60  0001 C CNN
 F 3 "" H 5200 -150 60  0000 C CNN
 F 4 "1, 4" V 2600 3750 60  0001 C CNN "CrossRef"
@@
 $EndComp
 $Comp
-L Device:R_Shunt RS11
+L Device:R RS11
 U 1 1 5AF1D15D
 P 10200 14900
 F 0 "RS11" V 10175 14495 60  0000 L BNN
 F 1 "0R02" V 10180 15070 60  0000 L BNN
-F 2 "" H 10600 14800 60  0001 C CNN
+F 2 "Resistor_SMD:R_0603_1608Metric" H 10600 14800 60  0001 C CNN
 F 3 "" H 10600 14800 60  0000 C CNN
 F 4 "9" V 2100 1600 60  0001 C CNN "CrossRef"
-F 5 "9" V 2100 1600 60  0001 C CNN "CrossRef"
-F 6 "1, 4" V 2100 1600 60  0001 C CNN "CrossRef"
-F 7 "1, 4" V 2100 1600 60  0001 C CNN "CrossRef"
-F 8 "1, 4" V 2100 1600 60  0001 C CNN "CrossRef"
-F 9 "" H 150 100 50  0001 C CNN "ClassName"
 	1    10200 14900
 	0    1    1    0
@@
 	10305 14500 11550 14500
 Wire Wire Line
-	9650 14900 10000 14900
-Wire Wire Line
-	10400 14900 10850 14900
-Wire Wire Line
-	10100 15050 10100 15200
-Wire Wire Line
-	10300 15050 10300 15100
-Wire Wire Line
-	10300 15100 11550 15100
-Wire Wire Line
 	4350 8500 4600 8500
 Wire Wire Line
@@
 NoConn ~ 11680 9500
 NoConn ~ 4600 9500
+Wire Wire Line
+	9650 14900 10050 14900
+Wire Wire Line
+	10350 14900 10850 14900
+Wire Wire Line
+	10050 14900 10050 15200
+Connection ~ 10050 14900
+Wire Wire Line
+	10350 14900 10350 15100
+Connection ~ 10350 14900
+Wire Wire Line
+	10350 15100 11550 15100
+Wire Wire Line
+	10050 15200 11550 15200
 Wire Bus Line
 	3450 3600 3450 3800
