File: kicad/DDR4_x8_32b_2_ECC-SchDoc.sch (KiCad schematic (older format))
At the start: 65 parts, among them U10 H5AN8G8NAFR-UH, U6 H5AN8G8NAFR-UH, U7 H5AN8G8NAFR-UH, U8 H5AN8G8NAFR-UH, U9 H5AN8G8NAFR-UH

Commit message: ki5 update
Parts:
- U10, U6, U7, U8, U9: footprint (none) -> Package_BGA:FBGA-78_7.5x11mm_Layout2x3x13_P0.8mm
Changed lines of the file:
@@
 EESchema Schematic File Version 4
-LIBS:Ki5-cache
 EELAYER 26 0
 EELAYER END
@@
 encoding utf-8
 Sheet 5 9
-Title "U540 RISC-V MPU eval board"
+Title "DDR4x8 32 Bit and ECC"
 Date "08 05 2018"
 Rev ""
 Comp ""
-Comment1 "DDR4x8 32 Bit and ECC"
+Comment1 ""
 Comment2 ""
 Comment3 ""
@@
 F 0 "U10" H 10705 13255 50  0000 C CNN
 F 1 "H5AN8G8NAFR-UH" H 11255 8645 50  0000 C CNN
-F 2 "" H 11260 6350 60  0001 C CNN
+F 2 "Package_BGA:FBGA-78_7.5x11mm_Layout2x3x13_P0.8mm" H 11260 6350 60  0001 C CNN
 F 3 "" H 11260 6350 60  0000 C CNN
 F 4 "" H 660 2250 50  0001 C CNN "ClassName"
@@
 F 0 "U9" H 4665 13250 50  0000 C CNN
 F 1 "H5AN8G8NAFR-UH" H 5245 8640 50  0000 C CNN
-F 2 "" H 5250 6350 60  0001 C CNN
+F 2 "Package_BGA:FBGA-78_7.5x11mm_Layout2x3x13_P0.8mm" H 5250 6350 60  0001 C CNN
 F 3 "" H 5250 6350 60  0000 C CNN
 F 4 "" H 650 2250 50  0001 C CNN "ClassName"
@@
 F 0 "U8" H 16365 7250 50  0000 C CNN
 F 1 "H5AN8G8NAFR-UH" H 16915 2635 50  0000 C CNN
-F 2 "" H 16945 350 60  0001 C CNN
+F 2 "Package_BGA:FBGA-78_7.5x11mm_Layout2x3x13_P0.8mm" H 16945 350 60  0001 C CNN
 F 3 "" H 16945 350 60  0000 C CNN
 F 4 "" H 645 2250 50  0001 C CNN "ClassName"
@@
 F 0 "U7" H 10575 7250 50  0000 C CNN
 F 1 "H5AN8G8NAFR-UH" H 11170 2640 50  0000 C CNN
-F 2 "" H 11155 350 60  0001 C CNN
+F 2 "Package_BGA:FBGA-78_7.5x11mm_Layout2x3x13_P0.8mm" H 11155 350 60  0001 C CNN
 F 3 "" H 11155 350 60  0000 C CNN
 F 4 "" H 655 2250 50  0001 C CNN "ClassName"
@@
 F 0 "U6" H 4680 7250 50  0000 C CNN
 F 1 "H5AN8G8NAFR-UH" H 5260 2635 50  0000 C CNN
-F 2 "" H 5255 350 60  0001 C CNN
+F 2 "Package_BGA:FBGA-78_7.5x11mm_Layout2x3x13_P0.8mm" H 5255 350 60  0001 C CNN
 F 3 "" H 5255 350 60  0000 C CNN
 F 4 "" H 655 2250 50  0001 C CNN "ClassName"
