File: kicad/Ki5.sch (KiCad schematic (older format))
At the start: 0 parts

Commit message: Ki5 update
Other:
- note added: "Ki5"
- note removed: "HiFive Unleashed"
Changed lines of the file:
@@
 EESchema Schematic File Version 4
-LIBS:HiFiveUnleashed-cache
+LIBS:Ki5-cache
 EELAYER 26 0
 EELAYER END
@@
 encoding utf-8
 Sheet 1 9
-Title ""
+Title "U540 RISC-V MPU eval board"
 Date ""
 Rev ""
@@
 F1 "Ethernet-SchDoc.sch" 50
 $EndSheet
-Text Notes 7250 7000 0    276  ~ 55
-HiFive Unleashed
+Text Notes 8735 7015 0    276  ~ 55
+Ki5
 Text Notes 800  1050 0    207  ~ 0
 Freedom U540 DDR and ChipLink
